Commit message: Add MoveIt Servo teleop: servo configs, launch, pose bridge

File: urdf_moveit/SH_Humanoid_v2_description/urdf/SH_Humanoid_v2.xacro (robot description, xacro)
@@ -309,5 +309,5 @@
   <child link="left_shoulder_pitch_link"/>
   <axis xyz="1.0 -0.000337 0.0"/>
-  <limit lower="-1.5708" upper="1.5708" effort="100" velocity="3.14"/>
+  <limit lower="-2.618" upper="2.618" effort="100" velocity="3.14"/>
 </joint>
 <joint name="left_shoulder_roll_joint" type="revolute">
@@ -316,5 +316,5 @@
   <child link="left_shoulder_roll_link"/>
   <axis xyz="-0.000337 -1.0 -0.000103"/>
-  <limit lower="-1.5708" upper="1.5708" effort="100" velocity="3.14"/>
+  <limit lower="-2.094" upper="2.094" effort="100" velocity="3.14"/>
 </joint>
 <joint name="left_shoulder_yaw_joint" type="revolute">
@@ -323,5 +323,5 @@
   <child link="left_shoulder_yaw_link"/>
   <axis xyz="-0.0 -0.000103 1.0"/>
-  <limit lower="-1.5708" upper="1.5708" effort="100" velocity="3.14"/>
+  <limit lower="-1.571" upper="1.571" effort="100" velocity="3.14"/>
 </joint>
 <joint name="left_elbow_joint" type="revolute">
@@ -330,5 +330,5 @@
   <child link="left_elbow_link"/>
   <axis xyz="-1.0 0.000337 0.0"/>
-  <limit lower="-1.5708" upper="1.5708" effort="100" velocity="3.14"/>
+  <limit lower="-2.618" upper="0.0" effort="100" velocity="3.14"/>
 </joint>
 <joint name="left_wrist_yaw_joint" type="revolute">
@@ -337,5 +337,5 @@
   <child link="left_wrist_yaw_link"/>
   <axis xyz="0.0 0.000103 -1.0"/>
-  <limit lower="-1.5708" upper="1.5708" effort="100" velocity="3.14"/>
+  <limit lower="-1.484" upper="1.484" effort="100" velocity="3.14"/>
 </joint>
 <joint name="left_wrist_pitch_joint" type="revolute">
@@ -344,5 +344,5 @@
   <child link="left_wrist_pitch_link"/>
   <axis xyz="0.000337 1.0 0.000103"/>
-  <limit lower="-1.5708" upper="1.5708" effort="100" velocity="3.14"/>
+  <limit lower="-1.396" upper="1.396" effort="100" velocity="3.14"/>
 </joint>
 <joint name="left_wrist_roll_joint" type="revolute">
@@ -351,5 +351,5 @@
   <child link="left_wrist_roll_link"/>
   <axis xyz="-1.0 0.000337 -0.0"/>
-  <limit lower="-1.5708" upper="1.5708" effort="100" velocity="3.14"/>
+  <limit lower="-1.571" upper="1.571" effort="100" velocity="3.14"/>
 </joint>
 <joint name="right_shoulder_pitch_joint" type="revolute">
@@ -358,5 +358,5 @@
   <child link="right_shoulder_pitch_link"/>
   <axis xyz="1.0 -0.000337 -0.0"/>
-  <limit lower="-1.5708" upper="1.5708" effort="100" velocity="3.14"/>
+  <limit lower="-2.618" upper="2.618" effort="100" velocity="3.14"/>
 </joint>
 <joint name="right_shoulder_roll_joint" type="revolute">
@@ -365,5 +365,5 @@
   <child link="right_shoulder_roll_link"/>
   <axis xyz="0.000337 1.0 0.000103"/>
-  <limit lower="-1.5708" upper="1.5708" effort="100" velocity="3.14"/>
+  <limit lower="-2.094" upper="2.094" effort="100" velocity="3.14"/>
 </joint>
 <joint name="right_shoulder_yaw_joint" type="revolute">
@@ -372,5 +372,5 @@
   <child link="right_shoulder_yaw_link"/>
   <axis xyz="0.0 0.000103 -1.0"/>
-  <limit lower="-1.5708" upper="1.5708" effort="100" velocity="3.14"/>
+  <limit lower="-1.571" upper="1.571" effort="100" velocity="3.14"/>
 </joint>
 <joint name="right_elbow_joint" type="revolute">
@@ -379,5 +379,5 @@
   <child link="right_elbow_link"/>
   <axis xyz="-1.0 0.000337 0.0"/>
-  <limit lower="-1.5708" upper="1.5708" effort="100" velocity="3.14"/>
+  <limit lower="-2.618" upper="0.0" effort="100" velocity="3.14"/>
 </joint>
 <joint name="right_wrist_yaw_joint" type="revolute">
@@ -386,5 +386,5 @@
   <child link="right_wrist_yaw_link"/>
   <axis xyz="0.0 -0.000103 1.0"/>
-  <limit lower="-1.5708" upper="1.5708" effort="100" velocity="3.14"/>
+  <limit lower="-1.484" upper="1.484" effort="100" velocity="3.14"/>
 </joint>
 <joint name="right_wrist_pitch_joint" type="revolute">
@@ -393,5 +393,5 @@
   <child link="right_wrist_pitch_link"/>
   <axis xyz="-0.000337 -1.0 -0.000103"/>
-  <limit lower="-1.5708" upper="1.5708" effort="100" velocity="3.14"/>
+  <limit lower="-1.396" upper="1.396" effort="100" velocity="3.14"/>
 </joint>
 <joint name="right_wrist_roll_joint" type="revolute">
@@ -400,5 +400,5 @@
   <child link="right_wrist_roll_link"/>
   <axis xyz="-1.0 0.000337 0.0"/>
-  <limit lower="-1.5708" upper="1.5708" effort="100" velocity="3.14"/>
+  <limit lower="-1.571" upper="1.571" effort="100" velocity="3.14"/>
 </joint>
   <link name="left_hand_link">
